File: guitar_dsp_platform.kicad_sch (KiCad schematic)
At the start: 0 parts

Commit message: Working on schematic
Other:
- sheet Analogue ports: added JACK_DETECT; removed AMP_DET, G_DET, PRE_IN_DET, PRE_OUT_DET
- sheet ESP32 ports: added JACK_DETECT; removed AMP_DET, G_DET, PRE_IN_DET, PRE_OUT_DET
