File: guitar_dsp_platform.kicad_sch (KiCad schematic)
At the start: 0 parts

Commit message: Ready for layout
Parts:
- added N101: 1598B, symbol Mechanical:Housing
Changed lines of the file:
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@@
     (stroke (width 0) (type solid) (color 0 0 0 0))
+  )
+  (symbol (lib_id "Mechanical:Housing") (at 168.91 62.23 0) (unit 1)
+    (in_bom yes) (on_board no) (fields_autoplaced)
+    (property "Reference" "N101" (id 0) (at 173.99 61.2774 0)
+      (effects (font (size 1.27 1.27)) (justify left))
+    )
+    (property "Value" "1598B" (id 1) (at 173.99 63.8174 0)
+      (effects (font (size 1.27 1.27)) (justify left))
+    )
+    (property "Footprint" "" (id 2) (at 170.18 60.96 0)
+      (effects (font (size 1.27 1.27)) hide)
+    )
+    (property "Datasheet" "https://www.mouser.co.uk/datasheet/2/177/1598-1389900.pdf" (id 3) (at 170.18 60.96 0)
+      (effects (font (size 1.27 1.27)) hide)
+    )
+    (property "PN" "1598BSGYPBK" (id 4) (at 168.91 62.23 0)
+      (effects (font (size 1.27 1.27)) hide)
+    )
   )
   (sheet (at 71.12 106.68) (size 16.51 30.48) (fields_autoplaced)
@@
     )
     (path "/00000000-0000-0000-0000-00005f70d2fd/00000000-0000-0000-0000-00005ffeb767"
-      (reference "L501") (unit 1) (value "22u") (footprint "")
+      (reference "L501") (unit 1) (value "22u") (footprint "Inductor_SMD:L_Taiyo-Yuden_NR-50xx_HandSoldering")
+    )
+    (path "/f174f29f-048a-478c-ae70-ff5265ccbc5a"
+      (reference "N101") (unit 1) (value "1598B") (footprint "")
     )
     (path "/00000000-0000-0000-0000-00005f70b353/7767c818-8af3-45a4-82d3-f66fb3d5e84c"

Commit message: Replace mounting holes with plated slots
Parts:
- added H101, H102, H103, H104, H105, H106: MountingHole, guitar_dsp_platform:1598B_mounting_hole, symbol Mechanical:MountingHole_Pad
Connections:
- new net GND: H101.1, H102.1, H103.1, H104.1, H105.1, H106.1
Changed lines of the file:
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@@
     (stroke (width 0) (type solid) (color 0 0 0 0))
+  )
+  (symbol (lib_id "power:GND") (at 189.23 53.34 0) (unit 1)
+    (in_bom yes) (on_board yes)
+    (property "Reference" "#PWR?" (id 0) (at 189.23 59.69 0)
+      (effects (font (size 1.27 1.27)) hide)
+    )
+    (property "Value" "GND" (id 1) (at 189.3316 57.277 0))
+    (property "Footprint" "" (id 2) (at 189.23 53.34 0)
+      (effects (font (size 1.27 1.27)) hide)
+    )
+    (property "Datasheet" "" (id 3) (at 189.23 53.34 0)
+      (effects (font (size 1.27 1.27)) hide)
+    )
+    (pin "1")
+  )
+  (symbol (lib_id "power:GND") (at 189.23 64.77 0) (unit 1)
+    (in_bom yes) (on_board yes)
+    (property "Reference" "#PWR?" (id 0) (at 189.23 71.12 0)
+      (effects (font (size 1.27 1.27)) hide)
+    )
+    (property "Value" "GND" (id 1) (at 189.3316 68.707 0))
+    (property "Footprint" "" (id 2) (at 189.23 64.77 0)
+      (effects (font (size 1.27 1.27)) hide)
+    )
+    (property "Datasheet" "" (id 3) (at 189.23 64.77 0)
+      (effects (font (size 1.27 1.27)) hide)
+    )
+    (pin "1")
+  )
+  (symbol (lib_id "power:GND") (at 189.23 76.2 0) (unit 1)
+    (in_bom yes) (on_board yes)
+    (property "Reference" "#PWR?" (id 0) (at 189.23 82.55 0)
+      (effects (font (size 1.27 1.27)) hide)
+    )
+    (property "Value" "GND" (id 1) (at 189.3316 80.137 0))
+    (property "Footprint" "" (id 2) (at 189.23 76.2 0)
+      (effects (font (size 1.27 1.27)) hide)
+    )
+    (property "Datasheet" "" (id 3) (at 189.23 76.2 0)
+      (effects (font (size 1.27 1.27)) hide)
+    )
+    (pin "1")
+  )
+  (symbol (lib_id "power:GND") (at 208.28 53.34 0) (unit 1)
+    (in_bom yes) (on_board yes)
+    (property "Reference" "#PWR?" (id 0) (at 208.28 59.69 0)
+      (effects (font (size 1.27 1.27)) hide)
+    )
+    (property "Value" "GND" (id 1) (at 208.3816 57.277 0))
+    (property "Footprint" "" (id 2) (at 208.28 53.34 0)
+      (effects (font (size 1.27 1.27)) hide)
+    )
+    (property "Datasheet" "" (id 3) (at 208.28 53.34 0)
+      (effects (font (size 1.27 1.27)) hide)
+    )
+    (pin "1")
+  )
+  (symbol (lib_id "power:GND") (at 208.28 64.77 0) (unit 1)
+    (in_bom yes) (on_board yes)
+    (property "Reference" "#PWR?" (id 0) (at 208.28 71.12 0)
+      (effects (font (size 1.27 1.27)) hide)
+    )
+    (property "Value" "GND" (id 1) (at 208.3816 68.707 0))
+    (property "Footprint" "" (id 2) (at 208.28 64.77 0)
+      (effects (font (size 1.27 1.27)) hide)
+    )
+    (property "Datasheet" "" (id 3) (at 208.28 64.77 0)
+      (effects (font (size 1.27 1.27)) hide)
+    )
+    (pin "1")
+  )
+  (symbol (lib_id "power:GND") (at 208.28 76.2 0) (unit 1)
+    (in_bom yes) (on_board yes)
+    (property "Reference" "#PWR?" (id 0) (at 208.28 82.55 0)
+      (effects (font (size 1.27 1.27)) hide)
+    )
+    (property "Value" "GND" (id 1) (at 208.3816 80.137 0))
+    (property "Footprint" "" (id 2) (at 208.28 76.2 0)
+      (effects (font (size 1.27 1.27)) hide)
+    )
+    (property "Datasheet" "" (id 3) (at 208.28 76.2 0)
+      (effects (font (size 1.27 1.27)) hide)
+    )
+    (pin "1")
+  )
+  (symbol (lib_id "Mechanical:MountingHole_Pad") (at 189.23 50.8 0) (unit 1)
+    (in_bom yes) (on_board yes)
+    (property "Reference" "H101" (id 0) (at 191.77 49.5299 0)
+      (effects (font (size 1.27 1.27)) (justify left))
+    )
+    (property "Value" "MountingHole" (id 1) (at 191.77 52.0699 0)
+      (effects (font (size 1.27 1.27)) (justify left))
+    )
+    (property "Footprint" "guitar_dsp_platform:1598B_mounting_hole" (id 2) (at 189.23 50.8 0)
+      (effects (font (size 1.27 1.27)) hide)
+    )
+    (property "Datasheet" "~" (id 3) (at 189.23 50.8 0)
+      (effects (font (size 1.27 1.27)) hide)
+    )
+    (pin "1")
+  )
+  (symbol (lib_id "Mechanical:MountingHole_Pad") (at 189.23 62.23 0) (unit 1)
+    (in_bom yes) (on_board yes) (fields_autoplaced)
+    (property "Reference" "H102" (id 0) (at 191.77 60.9599 0)
+      (effects (font (size 1.27 1.27)) (justify left))
+    )
+    (property "Value" "MountingHole" (id 1) (at 191.77 63.4999 0)
+      (effects (font (size 1.27 1.27)) (justify left))
+    )
+    (property "Footprint" "guitar_dsp_platform:1598B_mounting_hole" (id 2) (at 189.23 62.23 0)
+      (effects (font (size 1.27 1.27)) hide)
+    )
+    (property "Datasheet" "~" (id 3) (at 189.23 62.23 0)
+      (effects (font (size 1.27 1.27)) hide)
+    )
+    (pin "1")
+  )
+  (symbol (lib_id "Mechanical:MountingHole_Pad") (at 189.23 73.66 0) (unit 1)
+    (in_bom yes) (on_board yes) (fields_autoplaced)
+    (property "Reference" "H103" (id 0) (at 191.77 72.3899 0)
+      (effects (font (size 1.27 1.27)) (justify left))
+    )
+    (property "Value" "MountingHole" (id 1) (at 191.77 74.9299 0)
+      (effects (font (size 1.27 1.27)) (justify left))
+    )
+    (property "Footprint" "guitar_dsp_platform:1598B_mounting_hole" (id 2) (at 189.23 73.66 0)
+      (effects (font (size 1.27 1.27)) hide)
+    )
+    (property "Datasheet" "~" (id 3) (at 189.23 73.66 0)
+      (effects (font (size 1.27 1.27)) hide)
+    )
+    (pin "1")
+  )
+  (symbol (lib_id "Mechanical:MountingHole_Pad") (at 208.28 50.8 0) (unit 1)
+    (in_bom yes) (on_board yes) (fields_autoplaced)
+    (property "Reference" "H104" (id 0) (at 210.82 49.5299 0)
+      (effects (font (size 1.27 1.27)) (justify left))
+    )
+    (property "Value" "MountingHole" (id 1) (at 210.82 52.0699 0)
+      (effects (font (size 1.27 1.27)) (justify left))
+    )
+    (property "Footprint" "guitar_dsp_platform:1598B_mounting_hole" (id 2) (at 208.28 50.8 0)
+      (effects (font (size 1.27 1.27)) hide)
+    )
+    (property "Datasheet" "~" (id 3) (at 208.28 50.8 0)
+      (effects (font (size 1.27 1.27)) hide)
+    )
+    (pin "1")
+  )
+  (symbol (lib_id "Mechanical:MountingHole_Pad") (at 208.28 62.23 0) (unit 1)
+    (in_bom yes) (on_board yes) (fields_autoplaced)
+    (property "Reference" "H105" (id 0) (at 210.82 60.9599 0)
+      (effects (font (size 1.27 1.27)) (justify left))
+    )
+    (property "Value" "MountingHole" (id 1) (at 210.82 63.4999 0)
+      (effects (font (size 1.27 1.27)) (justify left))
+    )
+    (property "Footprint" "guitar_dsp_platform:1598B_mounting_hole" (id 2) (at 208.28 62.23 0)
+      (effects (font (size 1.27 1.27)) hide)
+    )
+    (property "Datasheet" "~" (id 3) (at 208.28 62.23 0)
+      (effects (font (size 1.27 1.27)) hide)
+    )
+    (pin "1")
+  )
+  (symbol (lib_id "Mechanical:MountingHole_Pad") (at 208.28 73.66 0) (unit 1)
+    (in_bom yes) (on_board yes) (fields_autoplaced)
+    (property "Reference" "H106" (id 0) (at 210.82 72.3899 0)
+      (effects (font (size 1.27 1.27)) (justify left))
+    )
+    (property "Value" "MountingHole" (id 1) (at 210.82 74.9299 0)
+      (effects (font (size 1.27 1.27)) (justify left))
+    )
+    (property "Footprint" "guitar_dsp_platform:1598B_mounting_hole" (id 2) (at 208.28 73.66 0)
+      (effects (font (size 1.27 1.27)) hide)
+    )
+    (property "Datasheet" "~" (id 3) (at 208.28 73.66 0)
+      (effects (font (size 1.27 1.27)) hide)
+    )
+    (pin "1")
   )
   (symbol (lib_id "Mechanical:Housing") (at 168.91 62.23 0) (unit 1)
@@
       (reference "#PWR0525") (unit 1) (value "+5V") (footprint "")
     )
+    (path "/0821d2ba-e74a-4062-a1ea-944c53fd8a9d"
+      (reference "#PWR?") (unit 1) (value "GND") (footprint "")
+    )
+    (path "/3cf9d353-21c3-48de-a571-d5a9ac825f8c"
+      (reference "#PWR?") (unit 1) (value "GND") (footprint "")
+    )
+    (path "/567f121b-d5f8-4886-8573-faa0b0050935"
+      (reference "#PWR?") (unit 1) (value "GND") (footprint "")
+    )
+    (path "/74c02de3-fb1c-4c01-8c98-9fd25e033326"
+      (reference "#PWR?") (unit 1) (value "GND") (footprint "")
+    )
+    (path "/77a38d5d-4947-4cda-84f8-64cba915d073"
+      (reference "#PWR?") (unit 1) (value "GND") (footprint "")
+    )
+    (path "/db3d1513-2929-41ae-9a3d-73b62e9ac3f6"
+      (reference "#PWR?") (unit 1) (value "GND") (footprint "")
+    )
     (path "/00000000-0000-0000-0000-00005fc20ef1/00000000-0000-0000-0000-00005feb8182"
       (reference "C201") (unit 1) (value "22u") (footprint "Capacitor_SMD:CP_Elec_4x5.8")
@@
       (reference "FB503") (unit 1) (value "1000R@100MHz") (footprint "Resistor_SMD:R_0805_2012Metric_Pad1.20x1.40mm_HandSolder")
     )
+    (path "/f940c2f2-c7cc-4935-ae7c-953db6379b8a"
+      (reference "H101") (unit 1) (value "MountingHole") (footprint "guitar_dsp_platform:1598B_mounting_hole")
+    )
+    (path "/79f525ed-db9a-47e5-b9e5-fa07c5ad75b4"
+      (reference "H102") (unit 1) (value "MountingHole") (footprint "guitar_dsp_platform:1598B_mounting_hole")
+    )
+    (path "/c89e7302-32d5-47c0-b8fe-9fcf68c9e9f3"
+      (reference "H103") (unit 1) (value "MountingHole") (footprint "guitar_dsp_platform:1598B_mounting_hole")
+    )
+    (path "/c7a15605-0ad6-4136-a73f-684c0bedb173"
+      (reference "H104") (unit 1) (value "MountingHole") (footprint "guitar_dsp_platform:1598B_mounting_hole")
+    )
+    (path "/24742546-c305-4837-84b4-09417022d295"
+      (reference "H105") (unit 1) (value "MountingHole") (footprint "guitar_dsp_platform:1598B_mounting_hole")
+    )
+    (path "/43556647-6c65-4070-91c7-434081da6987"
+      (reference "H106") (unit 1) (value "MountingHole") (footprint "guitar_dsp_platform:1598B_mounting_hole")
+    )
     (path "/00000000-0000-0000-0000-00005fc20ef1/00000000-0000-0000-0000-00005feb81a7"
