File: analogue.kicad_sch (KiCad schematic)
At the start: 72 parts, among them J201 NMJ6HCD2, J202 NMJ6HCD2, J203 NMJ6HCD2, J204 NMJ6HCD2, U201 OPA2197xD, U202 OPA2197xD, U203 OPA2197xD

Commit message: Working on schematic
Parts:
- removed C215, C222, C223: 100n, Capacitor_SMD:C_0805_2012Metric_Pad1.18x1.45mm_HandSolder, symbol Device:C_Small
- added R231, R234: 22k, Resistor_SMD:R_0805_2012Metric_Pad1.20x1.40mm_HandSolder, symbol Device:R_Small
- added R232: 10k, Resistor_SMD:R_0805_2012Metric_Pad1.20x1.40mm_HandSolder, symbol Device:R_Small
- added R233: 820, Resistor_SMD:R_0805_2012Metric_Pad1.20x1.40mm_HandSolder, symbol Device:R_Small
- R212, R228, R230: value 10k -> 820
- R219, R220, R229: value 10k -> 22k
Connections:
- net AMP_DET is gone; now on net VDD: R230.1
- net PRE_IN_DET is gone; now on net GND: R220.1
- net AMP_DET_JACK: now also R229.2; no longer R230.2
- net G_DET_JACK: now also R212.2; no longer R211.2
- net PRE_I_DET_JACK: now also R233.2, R234.2; no longer R212.2, R220.2
- net PRE_O_DET_JACK: now also R230.2, R231.2; no longer R227.2, R229.2
- net +3V3 renamed VDD
- net VDD: now also R233.1; no longer R211.1, R227.1
- net G_DET: no longer names the net of R219.1
- net G_DET: now also R220.2, R227.1; no longer C214.1
- net PRE_OUT_DET: no longer names the net of R229.1
- net PRE_OUT_DET: now also R211.1, R227.2
- new net: R211.2, R231.1, R232.1
- new net JACK_DETECT: C214.1, R232.2, R234.1
Other:
- moved on the sheet: R211

Commit message: Review PSU, add footprints for all components
Parts:
- R205, R206, R207, R208: value R -> DNF
- U201, U202, U203: PN (none) -> OPA2197ID
Connections:
- net AMP_DET_JACK: now also R212.2, R219.2; no longer R228.2, R229.2
- net G_DET_JACK: now also R233.2, R234.2; no longer R212.2, R219.2
- net PRE_I_DET_JACK: now also R228.2, R229.2; no longer R233.2, R234.2
Changed lines of the file:
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@@
     (stroke (width 0) (type solid) (color 0 0 0 0))
   )
-  (wire (pts (xy 172.72 133.35) (xy 185.42 133.35))
+  (wire (pts (xy 170.18 133.35) (xy 185.42 133.35))
     (stroke (width 0) (type solid) (color 0 0 0 0))
   )
@@
     (stroke (width 0) (type solid) (color 0 0 0 0))
   )
-  (wire (pts (xy 194.31 133.35) (xy 209.55 133.35))
+  (wire (pts (xy 193.04 133.35) (xy 209.55 133.35))
     (stroke (width 0) (type solid) (color 0 0 0 0))
   )
@@
     (stroke (width 0) (type solid) (color 0 0 0 0))
   )
-  (wire (pts (xy 248.92 133.35) (xy 265.43 133.35))
-    (stroke (width 0) (type solid) (color 0 0 0 0))
-  )
   (wire (pts (xy 252.73 36.83) (xy 260.35 36.83))
+    (stroke (width 0) (type solid) (color 0 0 0 0))
+  )
+  (wire (pts (xy 252.73 133.35) (xy 265.43 133.35))
     (stroke (width 0) (type solid) (color 0 0 0 0))
   )
@@
     (effects (font (size 1.27 1.27)) (justify left bottom))
   )
-  (label "G_DET_JACK" (at 172.72 133.35 0)
+  (label "AMP_DET_JACK" (at 170.18 133.35 0)
     (effects (font (size 1.27 1.27)) (justify left bottom))
   )
-  (label "AMP_DET_JACK" (at 194.31 133.35 0)
+  (label "PRE_I_DET_JACK" (at 193.04 133.35 0)
     (effects (font (size 1.27 1.27)) (justify left bottom))
   )
@@
     (effects (font (size 1.27 1.27)) (justify left bottom))
   )
-  (label "PRE_I_DET_JACK" (at 248.92 133.35 0)
+  (label "G_DET_JACK" (at 252.73 133.35 0)
     (effects (font (size 1.27 1.27)) (justify left bottom))
   )
@@
       (effects (font (size 1.27 1.27)) hide)
     )
+    (property "PN" "OPA2197ID" (id 4) (at 29.21 175.26 0)
+      (effects (font (size 1.27 1.27)) hide)
+    )
     (pin "4")
     (pin "8")
@@
       (effects (font (size 1.27 1.27)) hide)
     )
+    (property "PN" "OPA2197ID" (id 4) (at 48.26 175.26 0)
+      (effects (font (size 1.27 1.27)) hide)
+    )
     (pin "4")
     (pin "8")
@@
       (effects (font (size 1.27 1.27)) hide)
     )
+    (property "PN" "OPA2197ID" (id 4) (at 66.04 175.26 0)
+      (effects (font (size 1.27 1.27)) hide)
+    )
     (pin "4")
     (pin "8")
@@
       (effects (font (size 1.27 1.27)) (justify left))
     )
-    (property "Value" "R" (id 1) (at 94.488 151.003 0)
+    (property "Value" "DNF" (id 1) (at 94.488 151.003 0)
       (effects (font (size 1.27 1.27)) (justify left))
     )
@@
       (effects (font (size 1.27 1.27)) (justify left))
     )
-    (property "Value" "R" (id 1) (at 95.758 95.123 0)
+    (property "Value" "DNF" (id 1) (at 95.758 95.123 0)
       (effects (font (size 1.27 1.27)) (justify left))
     )
@@
     (in_bom yes) (on_board yes)
     (property "Reference" "R207" (id 0) (at 102.87 138.2522 90))
-    (property "Value" "R" (id 1) (at 102.87 140.5636 90))
+    (property "Value" "DNF" (id 1) (at 102.87 140.5636 90))
     (property "Footprint" "Resistor_SMD:R_0805_2012Metric_Pad1.20x1.40mm_HandSolder" (id 2) (at 102.87 141.732 90)
       (effects (font (size 1.27 1.27)) hide)
@@
     (in_bom yes) (on_board yes)
     (property "Reference" "R208" (id 0) (at 104.14 82.3722 90))
-    (property "Value" "R" (id 1) (at 104.14 84.6836 90))
+    (property "Value" "DNF" (id 1) (at 104.14 84.6836 90))
     (property "Footprint" "Resistor_SMD:R_0805_2012Metric_Pad1.20x1.40mm_HandSolder" (id 2) (at 104.14 85.852 90)
       (effects (font (size 1.27 1.27)) hide)
@@
       (effects (font (size 1.27 1.27)) hide)
     )
+    (property "PN" "OPA2197ID" (id 4) (at 62.23 25.4 0)
+      (effects (font (size 1.27 1.27)) hide)
+    )
     (pin "1")
     (pin "2")
@@
       (effects (font (size 1.27 1.27)) hide)
     )
+    (property "PN" "OPA2197ID" (id 4) (at 62.23 40.64 0)
+      (effects (font (size 1.27 1.27)) hide)
+    )
     (pin "5")
     (pin "6")
@@
       (effects (font (size 1.27 1.27)) hide)
     )
+    (property "PN" "OPA2197ID" (id 4) (at 101.6 120.65 0)
+      (effects (font (size 1.27 1.27)) hide)
+    )
     (pin "1")
     (pin "2")
@@
       (effects (font (size 1.27 1.27)) hide)
     )
+    (property "PN" "OPA2197ID" (id 4) (at 104.14 66.04 0)
+      (effects (font (size 1.27 1.27)) hide)
+    )
     (pin "1")
     (pin "2")
@@
       (effects (font (size 1.27 1.27)) hide)
     )
+    (property "PN" "OPA2197ID" (id 4) (at 227.33 36.83 0)
+      (effects (font (size 1.27 1.27)) hide)
+    )
     (pin "5")
     (pin "6")
@@
       (effects (font (size 1.27 1.27)) hide)
     )
+    (property "PN" "OPA2197ID" (id 4) (at 228.6 87.63 0)
+      (effects (font (size 1.27 1.27)) hide)
+    )

Commit message: Schematic reviewed, assign PN to all parts
Parts:
- R201, R202: PN (none) -> CR0805-FX-1004ELF
- R203, R204, R209, R210, R212, R221, R222, R223, R224, R228, R230, R233: PN (none) -> CR0805-FX-8200ELF
- R205, R206, R207, R208: value DNF -> TBD
- R211, R213, R214, R215, R216, R227, R232: PN (none) -> CR0805-FX-1002ELF
- R217, R218, R225, R226: PN (none) -> CR0805-FX-7501ELF
- R219, R220, R229, R231, R234: PN (none) -> CR0805-FX-2202ELF
- TP201, TP202, TP205, TP206: now left out of the parts list
Other:
- note removed: "Analogue"

Commit message: Start BOM tidy up
Parts:
- R201, R202, R205, R206, R207, R208, R209, R210: symbol Device:R -> Device:R_Small

Commit message: Update some part numbers for in-stock parts
Parts:
- C201: PN EEEFK1A220R -> EEEFK1A220AR
- D201, D202, D203, D204: value BAT54S -> BAS40-04; PN BAT54S -> BAS40-04,235
- FB201, FB202: value 600R@100MHz -> 1000R@100MHz; PN BLM21SP601SN1 -> 2508051027Y1
- R219, R220, R229, R231, R234: value 22k -> 20k; PN CR0805-FX-2202ELF -> CR0805-FX-2002ELF
- U201, U202, U203: value OPA2197xD -> OPA2156ID; PN OPA2197ID -> OPA2156ID

Commit message: Complete power supply design
Parts:
- C206, C207: symbol Device:C -> Device:C_Small
Connections:
- net at R208.1, R209.2, TP204.1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: no longer C207.1
- net at R206.1, R208.2, U201.2 (-): no longer C207.2
- net at R207.1, R210.2, TP203.1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: no longer C206.1
- net at R205.1, R207.2, U202.2 (-): no longer C206.2
Changed lines of the file:
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@@
+    (pin "2")
+  )
+  (symbol (lib_id "Device:C_Small") (at 102.87 133.35 270) (unit 1)
+    (in_bom yes) (on_board yes)
+    (property "Reference" "C206" (id 0) (at 102.87 126.9492 90))
+    (property "Value" "47p" (id 1) (at 102.87 129.2606 90))
+    (property "Footprint" "Capacitor_SMD:C_0805_2012Metric_Pad1.18x1.45mm_HandSolder" (id 2) (at 102.87 133.35 0)
+      (effects (font (size 1.27 1.27)) hide)
+    )
+    (property "Datasheet" "~" (id 3) (at 102.87 133.35 0)
+      (effects (font (size 1.27 1.27)) hide)
+    )
+    (property "PN" "885012007014" (id 4) (at 102.87 133.35 0)
+      (effects (font (size 1.27 1.27)) hide)
+    )
+    (pin "1")
+    (pin "2")
+  )
+  (symbol (lib_id "Device:C_Small") (at 104.14 77.47 270) (unit 1)
+    (in_bom yes) (on_board yes)
+    (property "Reference" "C207" (id 0) (at 104.14 71.0692 90))
+    (property "Value" "47p" (id 1) (at 104.14 73.3806 90))
+    (property "Footprint" "Capacitor_SMD:C_0805_2012Metric_Pad1.18x1.45mm_HandSolder" (id 2) (at 104.14 77.47 0)
+      (effects (font (size 1.27 1.27)) hide)
+    )
+    (property "Datasheet" "~" (id 3) (at 104.14 77.47 0)
+      (effects (font (size 1.27 1.27)) hide)
+    )
+    (property "PN" "885012007014" (id 4) (at 104.14 77.47 0)
+      (effects (font (size 1.27 1.27)) hide)
+    )
+    (pin "1")
     (pin "2")
   )
@@
       (effects (font (size 1.27 1.27)) hide)
     )
-    (pin "1")
-    (pin "2")
-  )
-  (symbol (lib_id "Device:C") (at 102.87 133.35 270) (unit 1)
-    (in_bom yes) (on_board yes)
-    (property "Reference" "C206" (id 0) (at 102.87 126.9492 90))
-    (property "Value" "47p" (id 1) (at 102.87 129.2606 90))
-    (property "Footprint" "Capacitor_SMD:C_0805_2012Metric_Pad1.18x1.45mm_HandSolder" (id 2) (at 99.06 134.3152 0)
-      (effects (font (size 1.27 1.27)) hide)
-    )
-    (property "Datasheet" "https://www.mouser.co.uk/datasheet/2/445/885012007014-1727155.pdf" (id 3) (at 102.87 133.35 0)
-      (effects (font (size 1.27 1.27)) hide)
-    )
-    (property "PN" "885012007014" (id 4) (at 102.87 133.35 0)
-      (effects (font (size 1.27 1.27)) hide)
-    )
-    (pin "1")
-    (pin "2")
-  )
-  (symbol (lib_id "Device:C") (at 104.14 77.47 270) (unit 1)
-    (in_bom yes) (on_board yes)
-    (property "Reference" "C207" (id 0) (at 104.14 71.0692 90))
-    (property "Value" "47p" (id 1) (at 104.14 73.3806 90))
-    (property "Footprint" "Capacitor_SMD:C_0805_2012Metric_Pad1.18x1.45mm_HandSolder" (id 2) (at 100.33 78.4352 0)
-      (effects (font (size 1.27 1.27)) hide)
-    )
-    (property "Datasheet" "https://www.mouser.co.uk/datasheet/2/445/885012007014-1727155.pdf" (id 3) (at 104.14 77.47 0)
-      (effects (font (size 1.27 1.27)) hide)
-    )
-    (property "PN" "885012007014" (id 4) (at 104.14 77.47 0)
-      (effects (font (size 1.27 1.27)) hide)
-    )

Commit message: Ready for layout
Connections:
- net at R208.1, R209.2, TP204.1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: now also C207.1
- net at R206.1, R208.2, U201.2 (-): now also C207.2
- net at R207.1, R210.2, TP203.1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: now also C206.1
- net at R205.1, R207.2, U202.2 (-): now also C206.2
Changed lines of the file:
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@@
+    (stroke (width 0) (type solid) (color 0 0 0 0))
+  )
+  (wire (pts (xy 92.71 133.35) (xy 100.33 133.35))
     (stroke (width 0) (type solid) (color 0 0 0 0))
   )
@@
     (stroke (width 0) (type solid) (color 0 0 0 0))
   )
+  (wire (pts (xy 93.98 77.47) (xy 101.6 77.47))
+    (stroke (width 0) (type solid) (color 0 0 0 0))
+  )
   (wire (pts (xy 93.98 87.63) (xy 93.98 91.44))
     (stroke (width 0) (type solid) (color 0 0 0 0))
@@
     (stroke (width 0) (type solid) (color 0 0 0 0))
   )
-  (wire (pts (xy 99.06 133.35) (xy 92.71 133.35))
-    (stroke (width 0) (type solid) (color 0 0 0 0))
-  )
-  (wire (pts (xy 100.33 77.47) (xy 93.98 77.47))
+  (wire (pts (xy 105.41 133.35) (xy 111.76 133.35))
     (stroke (width 0) (type solid) (color 0 0 0 0))
   )
@@
     (stroke (width 0) (type solid) (color 0 0 0 0))
   )
+  (wire (pts (xy 106.68 77.47) (xy 113.03 77.47))
+    (stroke (width 0) (type solid) (color 0 0 0 0))
+  )
   (wire (pts (xy 106.68 87.63) (xy 113.03 87.63))
-    (stroke (width 0) (type solid) (color 0 0 0 0))
-  )
-  (wire (pts (xy 106.68 133.35) (xy 111.76 133.35))
-    (stroke (width 0) (type solid) (color 0 0 0 0))
-  )
-  (wire (pts (xy 107.95 77.47) (xy 113.03 77.47))
     (stroke (width 0) (type solid) (color 0 0 0 0))
   )
@@
   )
   (symbol (lib_id "Device:C_Small") (at 102.87 133.35 270) (unit 1)
-    (in_bom yes) (on_board yes)
-    (property "Reference" "C206" (id 0) (at 102.87 126.9492 90))
-    (property "Value" "47p" (id 1) (at 102.87 129.2606 90))
+    (in_bom yes) (on_board yes) (fields_autoplaced)
+    (property "Reference" "C206" (id 0) (at 102.87 127 90))
+    (property "Value" "47p" (id 1) (at 102.87 129.54 90))
     (property "Footprint" "Capacitor_SMD:C_0805_2012Metric_Pad1.18x1.45mm_HandSolder" (id 2) (at 102.87 133.35 0)
       (effects (font (size 1.27 1.27)) hide)
@@
   )
   (symbol (lib_id "Device:C_Small") (at 104.14 77.47 270) (unit 1)
-    (in_bom yes) (on_board yes)
-    (property "Reference" "C207" (id 0) (at 104.14 71.0692 90))
-    (property "Value" "47p" (id 1) (at 104.14 73.3806 90))
+    (in_bom yes) (on_board yes) (fields_autoplaced)
+    (property "Reference" "C207" (id 0) (at 104.14 71.12 90))
+    (property "Value" "47p" (id 1) (at 104.14 73.66 90))
     (property "Footprint" "Capacitor_SMD:C_0805_2012Metric_Pad1.18x1.45mm_HandSolder" (id 2) (at 104.14 77.47 0)
       (effects (font (size 1.27 1.27)) hide)
