File: analogue.kicad_sch (KiCad schematic)
At the start: 73 parts, among them J201 NMJ6HCD2, J202 NMJ6HCD2, J203 NMJ6HCD2, J204 NMJ6HCD2, U201 OPA2156ID, U202 OPA2156ID, U203 OPA2156ID

Commit message: Final BOM changes
Parts:
- C210, C211, C220, C221: PN 865080640004 -> EEE1CA4R7NR
Changed lines of the file:
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@@
       (effects (font (size 1.27 1.27)) hide)
     )
-    (property "Datasheet" "https://www.mouser.co.uk/datasheet/2/445/865080640004-1726463.pdf" (id 3) (at 134.62 74.93 0)
+    (property "Datasheet" "https://industrial.panasonic.com/cdbs/www-data/pdf/RDE0000/ABA0000C1145.pdf" (id 3) (at 134.62 74.93 0)
       (effects (font (size 1.27 1.27)) hide)
     )
-    (property "PN" "865080640004" (id 4) (at 134.62 74.93 0)
+    (property "PN" "EEE1CA4R7NR" (id 4) (at 134.62 74.93 0)
       (effects (font (size 1.27 1.27)) hide)
     )
@@
       (effects (font (size 1.27 1.27)) hide)
     )
-    (property "Datasheet" "https://www.mouser.co.uk/datasheet/2/445/865080640004-1726463.pdf" (id 3) (at 134.62 129.54 0)
+    (property "Datasheet" "https://industrial.panasonic.com/cdbs/www-data/pdf/RDE0000/ABA0000C1145.pdf" (id 3) (at 134.62 129.54 0)
       (effects (font (size 1.27 1.27)) hide)
     )
-    (property "PN" "865080640004" (id 4) (at 134.62 129.54 0)
+    (property "PN" "EEE1CA4R7NR" (id 4) (at 134.62 129.54 0)
       (effects (font (size 1.27 1.27)) hide)
     )
@@
       (effects (font (size 1.27 1.27)) hide)
     )
-    (property "Datasheet" "https://www.mouser.co.uk/datasheet/2/445/865080640004-1726463.pdf" (id 3) (at 248.92 87.63 0)
+    (property "Datasheet" "https://industrial.panasonic.com/cdbs/www-data/pdf/RDE0000/ABA0000C1145.pdf" (id 3) (at 248.92 87.63 0)
       (effects (font (size 1.27 1.27)) hide)
     )
-    (property "PN" "865080640004" (id 4) (at 248.92 87.63 0)
+    (property "PN" "EEE1CA4R7NR" (id 4) (at 248.92 87.63 0)
       (effects (font (size 1.27 1.27)) hide)
     )
@@
       (effects (font (size 1.27 1.27)) hide)
     )
-    (property "Datasheet" "https://www.mouser.co.uk/datasheet/2/445/865080640004-1726463.pdf" (id 3) (at 250.19 36.83 0)
+    (property "Datasheet" "https://industrial.panasonic.com/cdbs/www-data/pdf/RDE0000/ABA0000C1145.pdf" (id 3) (at 250.19 36.83 0)
       (effects (font (size 1.27 1.27)) hide)
     )
-    (property "PN" "865080640004" (id 4) (at 250.19 36.83 0)
+    (property "PN" "EEE1CA4R7NR" (id 4) (at 250.19 36.83 0)
       (effects (font (size 1.27 1.27)) hide)
     )

Commit message: Tweak mechanical design
1/4 inch jacks are now flush with the faceplate. Reduced the gap between
MIDI jack and back faceplate.
Connections:
- net AMP_DET_JACK: now also R233.2, R234.2; no longer R212.2, R219.2
- net G_DET_JACK: now also R212.2, R219.2; no longer R233.2, R234.2
- net PRE_I_DET_JACK: now also R230.2, R231.2; no longer R228.2, R229.2
- net PRE_O_DET_JACK: now also R228.2, R229.2; no longer R230.2, R231.2
Changed lines of the file:
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@@
     (stroke (width 0) (type solid) (color 0 0 0 0))
   )
-  (wire (pts (xy 170.18 133.35) (xy 185.42 133.35))
+  (wire (pts (xy 172.72 133.35) (xy 185.42 133.35))
     (stroke (width 0) (type solid) (color 0 0 0 0))
   )
@@
     (stroke (width 0) (type solid) (color 0 0 0 0))
   )
+  (wire (pts (xy 191.77 133.35) (xy 209.55 133.35))
+    (stroke (width 0) (type solid) (color 0 0 0 0))
+  )
   (wire (pts (xy 193.04 69.85) (xy 223.52 69.85))
     (stroke (width 0) (type solid) (color 0 0 0 0))
@@
     (stroke (width 0) (type solid) (color 0 0 0 0))
   )
-  (wire (pts (xy 193.04 133.35) (xy 209.55 133.35))
-    (stroke (width 0) (type solid) (color 0 0 0 0))
-  )
   (wire (pts (xy 196.85 52.07) (xy 191.77 52.07))
     (stroke (width 0) (type solid) (color 0 0 0 0))
@@
     (stroke (width 0) (type solid) (color 0 0 0 0))
   )
+  (wire (pts (xy 250.19 133.35) (xy 265.43 133.35))
+    (stroke (width 0) (type solid) (color 0 0 0 0))
+  )
   (wire (pts (xy 252.73 36.83) (xy 260.35 36.83))
     (stroke (width 0) (type solid) (color 0 0 0 0))
   )
-  (wire (pts (xy 252.73 133.35) (xy 265.43 133.35))
-    (stroke (width 0) (type solid) (color 0 0 0 0))
-  )
   (wire (pts (xy 255.27 144.78) (xy 265.43 144.78))
     (stroke (width 0) (type solid) (color 0 0 0 0))
@@
     (effects (font (size 1.27 1.27)) (justify left bottom))
   )
-  (label "AMP_DET_JACK" (at 170.18 133.35 0)
-    (effects (font (size 1.27 1.27)) (justify left bottom))
-  )
-  (label "PRE_I_DET_JACK" (at 193.04 133.35 0)
+  (label "G_DET_JACK" (at 172.72 133.35 0)
+    (effects (font (size 1.27 1.27)) (justify left bottom))
+  )
+  (label "PRE_O_DET_JACK" (at 191.77 133.35 0)
     (effects (font (size 1.27 1.27)) (justify left bottom))
   )
@@
     (effects (font (size 1.27 1.27)) (justify right bottom))
   )
-  (label "PRE_O_DET_JACK" (at 219.71 133.35 0)
+  (label "PRE_I_DET_JACK" (at 219.71 133.35 0)
     (effects (font (size 1.27 1.27)) (justify left bottom))
   )
@@
     (effects (font (size 1.27 1.27)) (justify left bottom))
   )
-  (label "G_DET_JACK" (at 252.73 133.35 0)
-    (effects (font (size 1.27 1.27)) (justify left bottom))
-  )
+  (label "AMP_DET_JACK" (at 250.19 133.35 0)
+    (effects (font (size 1.27 1.27)) (justify left bottom))
+  )
