File: esp.kicad_sch (KiCad schematic)
At the start: 26 parts, among them J401 57PC5F, J402 57PC5F, J403 I2S testpoint, Q401 2N3904, U401 ESP32-DEVKIT-CVE, U402 6N138

Commit message: Working on schematic
Parts:
- R403, R406: footprint (none) -> Resistor_SMD:R_0805_2012Metric_Pad1.20x1.40mm_HandSolder
Connections:
- net +3V3 is gone; now on net VDD: R401.1
- net AMP_DET renamed I1
- net G_DET renamed JACK_DETECT
- net PRE_IN_DET renamed I3
- net PRE_OUT_DET renamed I2
- no-connect marks 25 -> 26
Other:
- note removed: "Jack detect signals"
Changed lines of the file:
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@@
   (no_connect (at 77.47 76.2))
   (no_connect (at 80.01 33.02))
+  (no_connect (at 80.01 38.1))
+  (no_connect (at 80.01 40.64))
   (no_connect (at 83.82 144.78))
   (no_connect (at 99.06 144.78))
@@
   (no_connect (at 137.16 53.34))
   (no_connect (at 137.16 55.88))
-  (no_connect (at 137.16 71.12))
-  (no_connect (at 137.16 73.66))
   (no_connect (at 137.16 78.74))
   (no_connect (at 137.16 81.28))
+  (no_connect (at 137.16 83.82))
   (no_connect (at 154.94 151.13))
   (no_connect (at 232.41 115.57))
@@
     (stroke (width 0) (type solid) (color 0 0 0 0))
   )
-  (wire (pts (xy 36.83 63.5) (xy 45.72 63.5))
-    (stroke (width 0) (type solid) (color 0 0 0 0))
-  )
-  (wire (pts (xy 36.83 66.04) (xy 45.72 66.04))
-    (stroke (width 0) (type solid) (color 0 0 0 0))
-  )
-  (wire (pts (xy 36.83 68.58) (xy 45.72 68.58))
-    (stroke (width 0) (type solid) (color 0 0 0 0))
-  )
-  (wire (pts (xy 36.83 71.12) (xy 45.72 71.12))
-    (stroke (width 0) (type solid) (color 0 0 0 0))
-  )
   (wire (pts (xy 49.53 177.8) (xy 35.56 177.8))
     (stroke (width 0) (type solid) (color 0 0 0 0))
@@
     (stroke (width 0) (type solid) (color 0 0 0 0))
   )
-  (wire (pts (xy 81.28 38.1) (xy 85.09 38.1))
-    (stroke (width 0) (type solid) (color 0 0 0 0))
-  )
-  (wire (pts (xy 81.28 40.64) (xy 85.09 40.64))
+  (wire (pts (xy 80.01 38.1) (xy 85.09 38.1))
+    (stroke (width 0) (type solid) (color 0 0 0 0))
+  )
+  (wire (pts (xy 80.01 40.64) (xy 85.09 40.64))
     (stroke (width 0) (type solid) (color 0 0 0 0))
   )
@@
     (stroke (width 0) (type solid) (color 0 0 0 0))
   )
-  (wire (pts (xy 115.57 71.12) (xy 137.16 71.12))
+  (wire (pts (xy 115.57 71.12) (xy 135.89 71.12))
     (stroke (width 0) (type solid) (color 0 0 0 0))
   )
@@
     (stroke (width 0) (type solid) (color 0 0 0 0))
   )
-  (wire (pts (xy 115.57 83.82) (xy 135.89 83.82))
+  (wire (pts (xy 115.57 83.82) (xy 137.16 83.82))
     (stroke (width 0) (type solid) (color 0 0 0 0))
   )
@@
     (stroke (width 0) (type solid) (color 0 0 0 0))
   )
+  (wire (pts (xy 135.89 73.66) (xy 115.57 73.66))
+    (stroke (width 0) (type solid) (color 0 0 0 0))
+  )
   (wire (pts (xy 137.16 66.04) (xy 115.57 66.04))
     (stroke (width 0) (type solid) (color 0 0 0 0))
@@
     (stroke (width 0) (type solid) (color 0 0 0 0))
   )
-  (wire (pts (xy 137.16 73.66) (xy 115.57 73.66))
-    (stroke (width 0) (type solid) (color 0 0 0 0))
-  )
   (wire (pts (xy 138.43 147.32) (xy 138.43 151.13))
     (stroke (width 0) (type solid) (color 0 0 0 0))
@@
     (stroke (width 0) (type solid) (color 0 0 0 0))
   )
-  (text "Jack detect signals" (at 26.67 59.69 0)
-    (effects (font (size 1.27 1.27)) (justify left bottom))
-  )
   (text "Internal flash interface" (at 63.5 59.69 0)
     (effects (font (size 1.27 1.27)) (justify left bottom))
   )
-  (text "INPUT ONLY" (at 80.01 38.1 180)
-    (effects (font (size 1.27 1.27)) (justify right bottom))
-  )
-  (text "INPUT ONLY" (at 80.01 40.64 180)
-    (effects (font (size 1.27 1.27)) (justify right bottom))
-  )
-  (text "INPUT ONLY" (at 137.16 83.82 0)
-    (effects (font (size 1.27 1.27)) (justify left bottom))
-  )
-  (text "INPUT ONLY" (at 137.16 86.36 0)
+  (text "INPUT ONLY" (at 78.74 38.1 180)
+    (effects (font (size 1.27 1.27)) (justify right bottom))
+  )
+  (text "INPUT ONLY" (at 78.74 40.64 180)
+    (effects (font (size 1.27 1.27)) (justify right bottom))
+  )
+  (text "INPUT ONLY" (at 115.57 83.82 0)
+    (effects (font (size 1.27 1.27)) (justify left bottom))
+  )
+  (text "INPUT ONLY" (at 115.57 86.36 0)
     (effects (font (size 1.27 1.27)) (justify left bottom))
   )
@@
     (effects (font (size 1.27 1.27)) (justify left bottom))
   )
-  (label "I0" (at 45.72 63.5 180)
-    (effects (font (size 1.27 1.27)) (justify right bottom))
-  )
-  (label "I1" (at 45.72 66.04 180)
-    (effects (font (size 1.27 1.27)) (justify right bottom))
-  )
-  (label "I2" (at 45.72 68.58 180)
-    (effects (font (size 1.27 1.27)) (justify right bottom))
-  )
-  (label "I3" (at 45.72 71.12 180)
-    (effects (font (size 1.27 1.27)) (justify right bottom))
-  )
   (label "SD0" (at 78.74 63.5 0)
     (effects (font (size 1.27 1.27)) (justify left bottom))
@@
     (effects (font (size 1.27 1.27)) (justify right bottom))
   )
-  (label "I0" (at 135.89 86.36 180)
-    (effects (font (size 1.27 1.27)) (justify right bottom))
-  )
   (label "MIDI_RX_uC" (at 176.53 156.21 180)
     (effects (font (size 1.27 1.27)) (justify right bottom))
@@
     (effects (font (size 1.27 1.27)) (justify right bottom))
   )
-  (hierarchical_label "G_DET" (shape input) (at 36.83 63.5 180)
-    (effects (font (size 1.27 1.27)) (justify right))
-  )
-  (hierarchical_label "AMP_DET" (shape input) (at 36.83 66.04 180)
-    (effects (font (size 1.27 1.27)) (justify right))
-  )
-  (hierarchical_label "PRE_OUT_DET" (shape input) (at 36.83 68.58 180)
-    (effects (font (size 1.27 1.27)) (justify right))
-  )
-  (hierarchical_label "PRE_IN_DET" (shape input) (at 36.83 71.12 180)
-    (effects (font (size 1.27 1.27)) (justify right))
+  (hierarchical_label "JACK_DETECT" (shape input) (at 135.89 86.36 0)
+    (effects (font (size 1.27 1.27)) (justify left))
   )
   (hierarchical_label "SDA" (shape tri_state) (at 137.16 66.04 0)
@@
     (effects (font (size 1.27 1.27)) (justify left))
   )
-  (symbol (lib_id "power:+3V3") (at 26.67 167.64 0) (unit 1)
-    (in_bom yes) (on_board yes)
-    (property "Reference" "#PWR0401" (id 0) (at 26.67 171.45 0)
-      (effects (font (size 1.27 1.27)) hide)
-    )
-    (property "Value" "+3V3" (id 1) (at 27.051 163.2458 0))
+  (symbol (lib_id "power:VDD") (at 26.67 167.64 0) (unit 1)
+    (in_bom yes) (on_board yes) (fields_autoplaced)
+    (property "Reference" "#PWR0103" (id 0) (at 26.67 171.45 0)
+      (effects (font (size 1.27 1.27)) hide)
+    )
+    (property "Value" "VDD" (id 1) (at 26.67 162.56 0))
     (property "Footprint" "" (id 2) (at 26.67 167.64 0)
       (effects (font (size 1.27 1.27)) hide)
@@
     (property "Reference" "R403" (id 0) (at 121.92 153.67 90))
     (property "Value" "220" (id 1) (at 121.92 156.21 90))
-    (property "Footprint" "" (id 2) (at 121.92 160.02 0)
+    (property "Footprint" "Resistor_SMD:R_0805_2012Metric_Pad1.20x1.40mm_HandSolder" (id 2) (at 121.92 160.02 0)
       (effects (font (size 1.27 1.27)) hide)
     )
@@
       (effects (font (size 1.27 1.27)) (justify left))
     )
-    (property "Footprint" "" (id 2) (at 212.09 123.19 0)
-      (effects (font (size 1.27 1.27)) hide)
-    )
+    (property "Footprint" "Resistor_SMD:R_0805_2012Metric_Pad1.20x1.40mm_HandSolder" (id 2) (at 212.09 123.19 0)
+      (effects (font (size 1.27 1.27)) hide)
+    )

Commit message: Review PSU, add footprints for all components
Parts:
- J401, J402: PN (none) -> 57PC5F
- Q401: PN (none) -> 2N3904
- R412: footprint (none) -> Resistor_SMD:R_1206_3216Metric_Pad1.30x1.75mm_HandSolder; PN (none) -> ESR18EZPF33R0
- U401: value ESP32-DEVKIT-CVE -> ESP32-DEVKITC-VE; PN (none) -> ESP32-DEVKITC-VE
- U402: PN (none) -> 6N138SDM
Changed lines of the file:
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@@
       (effects (font (size 1.27 1.27)) (justify left))
     )
-    (property "Footprint" "" (id 2) (at 254 113.03 0)
-      (effects (font (size 1.27 1.27)) hide)
-    )
-    (property "Datasheet" "~" (id 3) (at 254 113.03 0)
+    (property "Footprint" "Resistor_SMD:R_1206_3216Metric_Pad1.30x1.75mm_HandSolder" (id 2) (at 254 113.03 0)
+      (effects (font (size 1.27 1.27)) hide)
+    )
+    (property "Datasheet" "https://4donline.ihs.com/images/VipMasterIC/IC/ROHM/ROHM-S-A0011075102/ROHM-S-A0011075102-1.pdf?hkey=CECEF36DEECDED6468708AAF2E19C0C6" (id 3) (at 254 113.03 0)
+      (effects (font (size 1.27 1.27)) hide)
+    )
+    (property "PN" "ESR18EZPF33R0" (id 4) (at 254 113.03 0)
       (effects (font (size 1.27 1.27)) hide)
     )
@@
     (property "Datasheet" "https://www.onsemi.com/pub/Collateral/2N3903-D.PDF" (id 3) (at 209.55 133.35 0)
       (effects (font (size 1.27 1.27)) (justify left) hide)
+    )
+    (property "PN" "2N3904" (id 4) (at 209.55 133.35 0)
+      (effects (font (size 1.27 1.27)) hide)
     )
     (pin "1")
@@
       (effects (font (size 1.27 1.27)) hide)
     )
+    (property "PN" "57PC5F" (id 4) (at 91.44 144.78 0)
+      (effects (font (size 1.27 1.27)) hide)
+    )
     (pin "1")
     (pin "2")
@@
       (effects (font (size 1.27 1.27)) hide)
     )
+    (property "PN" "57PC5F" (id 4) (at 240.03 115.57 0)
+      (effects (font (size 1.27 1.27)) hide)
+    )
     (pin "1")
     (pin "2")
@@
       (effects (font (size 1.27 1.27)) hide)
     )
+    (property "PN" "6N138SDM" (id 4) (at 147.32 153.67 0)
+      (effects (font (size 1.27 1.27)) hide)
+    )
     (pin "1")
     (pin "2")
@@
     (in_bom yes) (on_board yes)
     (property "Reference" "U401" (id 0) (at 91.44 29.21 0))
-    (property "Value" "ESP32-DEVKIT-CVE" (id 1) (at 114.3 29.21 0))
+    (property "Value" "ESP32-DEVKITC-VE" (id 1) (at 114.3 29.21 0))
     (property "Footprint" "guitar_dsp_platform:ESP32_DevkitC" (id 2) (at 100.33 93.98 0)
       (effects (font (size 1.27 1.27)) hide)
@@
       (effects (font (size 1.27 1.27)) hide)
     )
+    (property "PN" "ESP32-DEVKITC-VE" (id 4) (at 100.33 63.5 0)
+      (effects (font (size 1.27 1.27)) hide)
+    )

Commit message: Schematic reviewed, assign PN to all parts
Parts:
- removed Q401: 2N3904, Package_TO_SOT_THT:TO-92_Inline, symbol Transistor_BJT:2N3904
- added C404: 100n, Capacitor_SMD:C_0805_2012Metric_Pad1.18x1.45mm_HandSolder, symbol Device:C_Small
- added D402: BAT760-7, Diode_SMD:D_SOD-323_HandSoldering, symbol Device:D_Schottky_Small
- added FB405: 600R@100MHz, Resistor_SMD:R_0805_2012Metric_Pad1.20x1.40mm_HandSolder, symbol Device:Ferrite_Bead_Small
- added Q401: MMBT3904, Package_TO_SOT_SMD:SOT-23, symbol Transistor_BJT:MMBT3904
- J403: value I2S testpoint -> I2S; now left out of the parts list
- R401, R402: now left out of the parts list
- R403: PN (none) -> CR0805-FX-2200ELF
- R404: PN (none) -> CR0805-FX-8200ELF
- R405: value 7.5k -> 820; PN (none) -> CR0805-FX-8200ELF
- R406: PN (none) -> CR0805-FX-10R0ELF
- R407, R408, R409, R410, R411: PN (none) -> CR0805-FX-33R0ELF
Connections:
- net GND: now also C404.2, Q401.2 (E)
- net at R405.1: now also Q401.1 (B)
- net at R406.2: now also Q401.3 (C)
- net +5V: no longer names the net of U401.19 (5V)
- net +5V: now also D402.1 (K)
- new net: C404.1, D402.2 (A), FB405.1
- new net +6V: FB405.2
Other:
- note added: "Diode allows USB to be used on devkit without damage. USB must be unplugged before power to the board is removed! It might be possible to remove D3 from the devkit to ensure the USB port can not power the ESP32."
- note added: "Series termination for I2S signals Drive strength 2 (20mA ~34R) Coplanar waveguide with ground plane, 0.25 W, 0.2 H, 0.3 S (62R) Based on JLCPCB 7628 stackup"
- note removed: "ESP32"
- note removed: "Series termination for I2S signals Drive strength 1 (10mA ~68R) Coplanar waveguide, 0.2 W, 1.6 H, 0.3 G (98R)"

Commit message: WIP
Parts:
- added R? (x2): 10k, Resistor_SMD:R_0805_2012Metric_Pad1.20x1.40mm_HandSolder, symbol Device:R_Small
Connections:
- net SCL: now also R?.2
- net SDA: now also R?.2
- net VDD: now also R?.1, R?.1
Other:
- note added: "Series termination for I2S signals Drive strength 2 (20mA ~34R) Coplanar waveguide with ground plane 0.25 W, 0.2 H, 0.3 S (62R) Based on JLCPCB 7628 stackup"
- note removed: "Series termination for I2S signals Drive strength 2 (20mA ~34R) Coplanar waveguide with ground plane, 0.25 W, 0.2 H, 0.3 S (62R) Based on JLCPCB 7628 stackup"
- moved on the sheet: J403, R407, R408, R409, R410, R411
