File: esp.kicad_sch (KiCad schematic)
At the start: 31 parts, among them J401 57PC5F, J402 57PC5F, J403 I2S, Q401 MMBT3904, U401 ESP32-DEVKITC-VE, U402 6N138

Commit message: Layout first draft
Parts:
- D402: value BAT760-7 -> SS16-HF; footprint Diode_SMD:D_SOD-323_HandSoldering -> Diode_SMD:D_SMA_Handsoldering; PN BAT760-7 -> SS16-HF
Changed lines of the file:
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@@
     (in_bom yes) (on_board yes) (fields_autoplaced)
     (property "Reference" "D402" (id 0) (at 81.28 13.97 0))
-    (property "Value" "BAT760-7" (id 1) (at 81.28 16.51 0))
-    (property "Footprint" "Diode_SMD:D_SOD-323_HandSoldering" (id 2) (at 81.28 20.32 90)
+    (property "Value" "SS16-HF" (id 1) (at 81.28 16.51 0))
+    (property "Footprint" "Diode_SMD:D_SMA_Handsoldering" (id 2) (at 81.28 20.32 90)
       (effects (font (size 1.27 1.27)) hide)
     )
-    (property "Datasheet" "https://www.diodes.com/assets/Datasheets/ds30498.pdf" (id 3) (at 81.28 20.32 90)
+    (property "Datasheet" "https://www.mouser.co.uk/datasheet/2/80/20190514095348-2504793.pdf" (id 3) (at 81.28 20.32 90)
       (effects (font (size 1.27 1.27)) hide)
     )
-    (property "PN" "BAT760-7" (id 4) (at 81.28 20.32 0)
+    (property "PN" "SS16-HF" (id 4) (at 81.28 20.32 0)
       (effects (font (size 1.27 1.27)) hide)
     )

Commit message: Final BOM changes
Parts:
- Q401: PN MMBT3904LT1XT -> MMBT3904-G
Changed lines of the file:
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@@
       (effects (font (size 1.27 1.27) italic) (justify left) hide)
     )
-    (property "Datasheet" "https://www.onsemi.com/pub/Collateral/2N3903-D.PDF" (id 3) (at 209.55 133.35 0)
+    (property "Datasheet" "https://www.mouser.co.uk/datasheet/2/80/MMBT3904_G_RevE-2506519.pdf" (id 3) (at 209.55 133.35 0)
       (effects (font (size 1.27 1.27)) (justify left) hide)
     )
-    (property "PN" "MMBT3904LT1XT" (id 4) (at 209.55 133.35 0)
+    (property "PN" "MMBT3904-G" (id 4) (at 209.55 133.35 0)
       (effects (font (size 1.27 1.27)) hide)
     )

Commit message: Resolve some issues
- Add missing MIDI connector pins to symbol
- Isolate low-ESR capacitors from 1117
- Fix DRC errors in footprints
Parts:
- added C405: 100n, Capacitor_SMD:C_0805_2012Metric_Pad1.18x1.45mm_HandSolder, symbol Device:C_Small
- added R415: 0, Resistor_SMD:R_0805_2012Metric_Pad1.20x1.40mm_HandSolder, symbol Device:R_Small
- J401, J402: symbol Connector:DIN-5_180degree -> symbols:57PC5F
Connections:
- net GND: now also C405.2, R415.2
- new net: C405.1, J401.6, J401.7
- new net: J402.6, J402.7, R415.1
Changed lines of the file:
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@@
   (paper "A4")
   (junction (at 69.85 20.32) (diameter 0) (color 0 0 0 0))
+  (junction (at 91.44 176.53) (diameter 0) (color 0 0 0 0))
   (junction (at 93.98 20.32) (diameter 0) (color 0 0 0 0))
   (junction (at 157.48 148.59) (diameter 0.9144) (color 0 0 0 0))
   (junction (at 157.48 156.21) (diameter 0.9144) (color 0 0 0 0))
+  (junction (at 240.03 132.08) (diameter 0) (color 0 0 0 0))
   (junction (at 252.73 68.58) (diameter 0.9144) (color 0 0 0 0))
   (junction (at 252.73 71.12) (diameter 0.9144) (color 0 0 0 0))
@@
     (stroke (width 0) (type solid) (color 0 0 0 0))
   )
+  (wire (pts (xy 91.44 176.53) (xy 91.44 175.26))
+    (stroke (width 0) (type default) (color 0 0 0 0))
+  )
+  (wire (pts (xy 91.44 177.8) (xy 91.44 176.53))
+    (stroke (width 0) (type default) (color 0 0 0 0))
+  )
   (wire (pts (xy 93.98 19.05) (xy 93.98 20.32))
     (stroke (width 0) (type solid) (color 0 0 0 0))
@@
     (stroke (width 0) (type solid) (color 0 0 0 0))
   )
+  (wire (pts (xy 95.25 152.4) (xy 95.25 170.18))
+    (stroke (width 0) (type solid) (color 0 0 0 0))
+  )
+  (wire (pts (xy 95.25 175.26) (xy 95.25 176.53))
+    (stroke (width 0) (type default) (color 0 0 0 0))
+  )
+  (wire (pts (xy 95.25 176.53) (xy 91.44 176.53))
+    (stroke (width 0) (type default) (color 0 0 0 0))
+  )
   (wire (pts (xy 99.06 20.32) (xy 99.06 27.94))
     (stroke (width 0) (type solid) (color 0 0 0 0))
@@
     (stroke (width 0) (type solid) (color 0 0 0 0))
   )
+  (wire (pts (xy 240.03 132.08) (xy 240.03 123.19))
+    (stroke (width 0) (type default) (color 0 0 0 0))
+  )
+  (wire (pts (xy 240.03 132.08) (xy 243.84 132.08))
+    (stroke (width 0) (type default) (color 0 0 0 0))
+  )
+  (wire (pts (xy 240.03 133.35) (xy 240.03 132.08))
+    (stroke (width 0) (type default) (color 0 0 0 0))
+  )
   (wire (pts (xy 242.57 22.86) (xy 257.81 22.86))
     (stroke (width 0) (type solid) (color 0 0 0 0))
@@
   (wire (pts (xy 242.57 53.34) (xy 257.81 53.34))
     (stroke (width 0) (type solid) (color 0 0 0 0))
+  )
+  (wire (pts (xy 243.84 123.19) (xy 243.84 125.73))
+    (stroke (width 0) (type default) (color 0 0 0 0))
+  )
+  (wire (pts (xy 243.84 132.08) (xy 243.84 130.81))
+    (stroke (width 0) (type default) (color 0 0 0 0))
   )
   (wire (pts (xy 247.65 118.11) (xy 254 118.11))
@@
     (pin "1")
   )
-  (symbol (lib_id "power:GND") (at 91.44 175.26 0) (unit 1)
-    (in_bom yes) (on_board yes)
-    (property "Reference" "#PWR0403" (id 0) (at 91.44 181.61 0)
-      (effects (font (size 1.27 1.27)) hide)
-    )
-    (property "Value" "GND" (id 1) (at 91.567 179.6542 0))
-    (property "Footprint" "" (id 2) (at 91.44 175.26 0)
-      (effects (font (size 1.27 1.27)) hide)
-    )
-    (property "Datasheet" "" (id 3) (at 91.44 175.26 0)
+  (symbol (lib_id "power:GND") (at 91.44 177.8 0) (unit 1)
+    (in_bom yes) (on_board yes)
+    (property "Reference" "#PWR0403" (id 0) (at 91.44 184.15 0)
+      (effects (font (size 1.27 1.27)) hide)
+    )
+    (property "Value" "GND" (id 1) (at 91.567 182.1942 0))
+    (property "Footprint" "" (id 2) (at 91.44 177.8 0)
+      (effects (font (size 1.27 1.27)) hide)
+    )
+    (property "Datasheet" "" (id 3) (at 91.44 177.8 0)
       (effects (font (size 1.27 1.27)) hide)
     )
@@
     (pin "1")
   )
-  (symbol (lib_id "power:GND") (at 240.03 123.19 0) (unit 1)
-    (in_bom yes) (on_board yes)
-    (property "Reference" "#PWR0412" (id 0) (at 240.03 129.54 0)
-      (effects (font (size 1.27 1.27)) hide)
-    )
-    (property "Value" "GND" (id 1) (at 240.157 127.5842 0))
-    (property "Footprint" "" (id 2) (at 240.03 123.19 0)
-      (effects (font (size 1.27 1.27)) hide)
-    )
-    (property "Datasheet" "" (id 3) (at 240.03 123.19 0)
+  (symbol (lib_id "power:GND") (at 240.03 133.35 0) (unit 1)
+    (in_bom yes) (on_board yes)
+    (property "Reference" "#PWR0412" (id 0) (at 240.03 139.7 0)
+      (effects (font (size 1.27 1.27)) hide)
+    )
+    (property "Value" "GND" (id 1) (at 240.157 137.7442 0))
+    (property "Footprint" "" (id 2) (at 240.03 133.35 0)
+      (effects (font (size 1.27 1.27)) hide)
+    )
+    (property "Datasheet" "" (id 3) (at 240.03 133.35 0)
       (effects (font (size 1.27 1.27)) hide)
     )
@@
     (pin "2")
   )
+  (symbol (lib_id "Device:R_Small") (at 243.84 128.27 0) (unit 1)
+    (in_bom yes) (on_board yes)
+    (property "Reference" "R415" (id 0) (at 245.3386 127.1016 0)
+      (effects (font (size 1.27 1.27)) (justify left))
+    )
+    (property "Value" "0" (id 1) (at 245.3386 129.413 0)
+      (effects (font (size 1.27 1.27)) (justify left))
+    )
+    (property "Footprint" "Resistor_SMD:R_0805_2012Metric_Pad1.20x1.40mm_HandSolder" (id 2) (at 243.84 128.27 0)
+      (effects (font (size 1.27 1.27)) hide)
+    )
+    (property "Datasheet" "~" (id 3) (at 243.84 128.27 0)
+      (effects (font (size 1.27 1.27)) hide)
+    )
+    (property "PN" "CR0805-J/-000ELF" (id 4) (at 243.84 128.27 0)
+      (effects (font (size 1.27 1.27)) hide)
+    )
+    (pin "1")
+    (pin "2")
+  )
   (symbol (lib_id "Device:R_Small") (at 254 113.03 0) (unit 1)
     (in_bom yes) (on_board yes) (fields_autoplaced)
@@
     (pin "2")
   )
-  (symbol (lib_id "Device:C_Small") (at 91.44 172.72 0) (unit 1)
-    (in_bom yes) (on_board yes)
-    (property "Reference" "C401" (id 0) (at 93.7768 171.5516 0)
-      (effects (font (size 1.27 1.27)) (justify left))
-    )
-    (property "Value" "100n" (id 1) (at 93.7768 173.863 0)
+  (symbol (lib_id "Device:C_Small") (at 91.44 172.72 0) (mirror y) (unit 1)
+    (in_bom yes) (on_board yes)
+    (property "Reference" "C401" (id 0) (at 89.1032 171.5516 0)
+      (effects (font (size 1.27 1.27)) (justify left))
+    )
+    (property "Value" "100n" (id 1) (at 89.1032 173.863 0)
       (effects (font (size 1.27 1.27)) (justify left))
     )
@@
     )
     (property "PN" "C0805C104M3RACTU" (id 4) (at 91.44 172.72 0)
+      (effects (font (size 1.27 1.27)) hide)
+    )
+    (pin "1")
+    (pin "2")
+  )
+  (symbol (lib_id "Device:C_Small") (at 95.25 172.72 0) (unit 1)
+    (in_bom yes) (on_board yes)
+    (property "Reference" "C405" (id 0) (at 97.5868 171.5516 0)
+      (effects (font (size 1.27 1.27)) (justify left))
+    )
+    (property "Value" "100n" (id 1) (at 97.5868 173.863 0)
+      (effects (font (size 1.27 1.27)) (justify left))
+    )
+    (property "Footprint" "Capacitor_SMD:C_0805_2012Metric_Pad1.18x1.45mm_HandSolder" (id 2) (at 95.25 172.72 0)
+      (effects (font (size 1.27 1.27)) hide)
+    )
+    (property "Datasheet" "https://www.mouser.co.uk/datasheet/2/212/KEM_C1002_X7R_SMD-1102033.pdf" (id 3) (at 95.25 172.72 0)
+      (effects (font (size 1.27 1.27)) hide)
+    )
+    (property "PN" "C0805C104M3RACTU" (id 4) (at 95.25 172.72 0)
       (effects (font (size 1.27 1.27)) hide)
     )
@@
     (pin "9")
   )
-  (symbol (lib_id "Connector:DIN-5_180degree") (at 91.44 144.78 180) (unit 1)
+  (symbol (lib_id "symbols:57PC5F") (at 91.44 144.78 180) (unit 1)
     (in_bom yes) (on_board yes) (fields_autoplaced)
     (property "Reference" "J401" (id 0) (at 91.44 134.62 0))
     (property "Value" "57PC5F" (id 1) (at 91.44 137.16 0))
-    (property "Footprint" "guitar_dsp_platform:57PC5F" (id 2) (at 91.44 144.78 0)
-      (effects (font (size 1.27 1.27)) hide)
-    )
-    (property "Datasheet" "http://www.mouser.com/ds/2/18/40_c091_abd_e-75918.pdf" (id 3) (at 91.44 144.78 0)
-      (effects (font (size 1.27 1.27)) hide)
-    )
-    (property "PN" "57PC5F" (id 4) (at 91.44 144.78 0)
+    (property "Footprint" "guitar_dsp_platform:57PC5F" (id 2) (at 91.44 134.62 0)
+      (effects (font (size 1.27 1.27)) hide)
+    )
+    (property "Datasheet" "https://www.mouser.co.uk/datasheet/2/393/57PC5F_CD-478737.pdf" (id 3) (at 91.44 137.16 0)
+      (effects (font (size 1.27 1.27)) hide)
+    )
+    (property "PN" "57PC5F" (id 4) (at 91.44 132.08 0)
       (effects (font (size 1.27 1.27)) hide)
     )
@@
     (pin "4")
     (pin "5")
-  )
-  (symbol (lib_id "Connector:DIN-5_180degree") (at 240.03 115.57 180) (unit 1)
+    (pin "6")
+    (pin "7")
+  )
+  (symbol (lib_id "symbols:57PC5F") (at 240.03 115.57 180) (unit 1)
     (in_bom yes) (on_board yes) (fields_autoplaced)
     (property "Reference" "J402" (id 0) (at 240.03 105.41 0))
     (property "Value" "57PC5F" (id 1) (at 240.03 107.95 0))
-    (property "Footprint" "guitar_dsp_platform:57PC5F" (id 2) (at 240.03 115.57 0)
-      (effects (font (size 1.27 1.27)) hide)
-    )
-    (property "Datasheet" "http://www.mouser.com/ds/2/18/40_c091_abd_e-75918.pdf" (id 3) (at 240.03 115.57 0)
-      (effects (font (size 1.27 1.27)) hide)
-    )
-    (property "PN" "57PC5F" (id 4) (at 240.03 115.57 0)
+    (property "Footprint" "guitar_dsp_platform:57PC5F" (id 2) (at 240.03 105.41 0)
+      (effects (font (size 1.27 1.27)) hide)
+    )
+    (property "Datasheet" "https://www.mouser.co.uk/datasheet/2/393/57PC5F_CD-478737.pdf" (id 3) (at 240.03 107.95 0)
+      (effects (font (size 1.27 1.27)) hide)
+    )
+    (property "PN" "57PC5F" (id 4) (at 240.03 102.87 0)
       (effects (font (size 1.27 1.27)) hide)
     )
@@
     (pin "4")
     (pin "5")
+    (pin "6")
+    (pin "7")
   )
   (symbol (lib_id "Isolator:6N138") (at 147.32 153.67 0) (unit 1)
