File: codec.kicad_sch (KiCad schematic)
At the start: 10 parts, among them U301 PCM3060

Commit message: Resolve some issues
- Add missing MIDI connector pins to symbol
- Isolate low-ESR capacitors from 1117
- Fix DRC errors in footprints
Parts:
- added NT301: Net-Tie_2, NetTie:NetTie-2_SMD_Pad0.5mm, symbol Device:Net-Tie_2
Connections:
- net GND: now also NT301.1; no longer U301.28 (MODE)
- new net MODE: NT301.2, U301.28 (MODE)
Other:
- moved on the sheet: R303
Changed lines of the file:
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@@
   (junction (at 147.32 69.85) (diameter 0.9144) (color 0 0 0 0))
   (junction (at 163.83 124.46) (diameter 0.9144) (color 0 0 0 0))
-  (junction (at 170.18 113.03) (diameter 0.9144) (color 0 0 0 0))
+  (junction (at 176.53 113.03) (diameter 0.9144) (color 0 0 0 0))
   (no_connect (at 153.67 100.33))
   (no_connect (at 153.67 102.87))
@@
     (stroke (width 0) (type solid) (color 0 0 0 0))
   )
-  (wire (pts (xy 146.05 113.03) (xy 170.18 113.03))
-    (stroke (width 0) (type solid) (color 0 0 0 0))
+  (wire (pts (xy 146.05 113.03) (xy 176.53 113.03))
+    (stroke (width 0) (type default) (color 0 0 0 0))
   )
   (wire (pts (xy 146.05 115.57) (xy 163.83 115.57))
@@
     (stroke (width 0) (type solid) (color 0 0 0 0))
   )
-  (wire (pts (xy 163.83 115.57) (xy 163.83 124.46))
+  (wire (pts (xy 163.83 115.57) (xy 163.83 116.84))
+    (stroke (width 0) (type solid) (color 0 0 0 0))
+  )
+  (wire (pts (xy 163.83 121.92) (xy 163.83 124.46))
     (stroke (width 0) (type solid) (color 0 0 0 0))
   )
@@
     (stroke (width 0) (type solid) (color 0 0 0 0))
   )
-  (wire (pts (xy 163.83 124.46) (xy 170.18 124.46))
-    (stroke (width 0) (type solid) (color 0 0 0 0))
-  )
-  (wire (pts (xy 170.18 113.03) (xy 170.18 115.57))
-    (stroke (width 0) (type solid) (color 0 0 0 0))
-  )
-  (wire (pts (xy 170.18 113.03) (xy 173.99 113.03))
-    (stroke (width 0) (type solid) (color 0 0 0 0))
-  )
-  (wire (pts (xy 170.18 120.65) (xy 170.18 124.46))
+  (wire (pts (xy 163.83 124.46) (xy 176.53 124.46))
+    (stroke (width 0) (type solid) (color 0 0 0 0))
+  )
+  (wire (pts (xy 176.53 113.03) (xy 176.53 115.57))
+    (stroke (width 0) (type solid) (color 0 0 0 0))
+  )
+  (wire (pts (xy 176.53 113.03) (xy 180.34 113.03))
+    (stroke (width 0) (type solid) (color 0 0 0 0))
+  )
+  (wire (pts (xy 176.53 120.65) (xy 176.53 124.46))
     (stroke (width 0) (type solid) (color 0 0 0 0))
   )
@@
     (effects (font (size 1.27 1.27)) (justify left))
   )
-  (hierarchical_label "~{RST}" (shape input) (at 173.99 113.03 0)
+  (hierarchical_label "~{RST}" (shape input) (at 180.34 113.03 0)
     (effects (font (size 1.27 1.27)) (justify left))
   )
@@
     )
     (pin "1")
+  )
+  (symbol (lib_id "Device:Net-Tie_2") (at 163.83 119.38 90) (unit 1)
+    (in_bom yes) (on_board yes) (fields_autoplaced)
+    (property "Reference" "NT301" (id 0) (at 165.1 119.3799 90)
+      (effects (font (size 1.27 1.27)) (justify right))
+    )
+    (property "Value" "Net-Tie_2" (id 1) (at 165.1 120.6499 90)
+      (effects (font (size 1.27 1.27)) (justify right) hide)
+    )
+    (property "Footprint" "NetTie:NetTie-2_SMD_Pad0.5mm" (id 2) (at 163.83 119.38 0)
+      (effects (font (size 1.27 1.27)) hide)
+    )
+    (property "Datasheet" "~" (id 3) (at 163.83 119.38 0)
+      (effects (font (size 1.27 1.27)) hide)
+    )
+    (pin "1")
+    (pin "2")
   )
   (symbol (lib_id "Connector:TestPoint") (at 85.09 101.6 0) (mirror y) (unit 1)
@@
     (pin "2")
   )
-  (symbol (lib_id "Device:R_Small") (at 170.18 118.11 0) (unit 1)
-    (in_bom yes) (on_board yes)
-    (property "Reference" "R303" (id 0) (at 171.6786 116.9416 0)
-      (effects (font (size 1.27 1.27)) (justify left))
-    )
-    (property "Value" "10k" (id 1) (at 171.6786 119.253 0)
-      (effects (font (size 1.27 1.27)) (justify left))
-    )
-    (property "Footprint" "Resistor_SMD:R_0805_2012Metric_Pad1.20x1.40mm_HandSolder" (id 2) (at 170.18 118.11 0)
-      (effects (font (size 1.27 1.27)) hide)
-    )
-    (property "Datasheet" "~" (id 3) (at 170.18 118.11 0)
-      (effects (font (size 1.27 1.27)) hide)
-    )
-    (property "PN" "CR0805-FX-1002ELF" (id 4) (at 170.18 118.11 0)
-      (effects (font (size 1.27 1.27)) hide)
-    )
+  (symbol (lib_id "Device:R_Small") (at 176.53 118.11 0) (unit 1)
+    (in_bom yes) (on_board yes)
+    (property "Reference" "R303" (id 0) (at 178.0286 116.9416 0)
+      (effects (font (size 1.27 1.27)) (justify left))
+    )
+    (property "Value" "10k" (id 1) (at 178.0286 119.253 0)
+      (effects (font (size 1.27 1.27)) (justify left))
+    )
+    (property "Footprint" "Resistor_SMD:R_0805_2012Metric_Pad1.20x1.40mm_HandSolder" (id 2) (at 176.53 118.11 0)
+      (effects (font (size 1.27 1.27)) hide)
+    )
+    (property "Datasheet" "~" (id 3) (at 176.53 118.11 0)
+      (effects (font (size 1.27 1.27)) hide)
+    )
+    (property "PN" "CR0805-FX-1002ELF" (id 4) (at 176.53 118.11 0)
+      (effects (font (size 1.27 1.27)) hide)
+    )
